Commit message: added launch files for aws

File: t2rgb_description/urdf/optimized/optimized_2023_05_17-03_42_06_PM.urdf.xacro (robot description, xacro)
@@ -23,5 +23,5 @@
   </gazebo>
   <joint name="camera_right_rgb_joint" type="fixed">
-    <origin xyz="0.003084837483015066 -0.03862858109122667 0.0012045523690927724" rpy="-0.019012904568392552 -0.007012354017393246 0.0044708591364499475"/>
+    <origin xyz="0.002729579820923045 -0.036125025053185524 0.0006995612951252911" rpy="0.005003475126905138 -0.0009618522961942883 0.004449245330954742"/>
     <parent link="camera_right_link"/>
     <child link="camera_right_rgb_frame"/>
@@ -111,5 +111,5 @@
   </gazebo>
   <joint name="camera_left_rgb_joint" type="fixed">
-    <origin xyz="0.0016748091127418792 -0.03814222599406782 -0.006507520212859007" rpy="-0.01895612012487999 -0.007321106971785336 0.003858542386210276"/>
+    <origin xyz="0.0006031919917758765 -0.03664342569680844 0.004645103530296592" rpy="0.005018998201366674 0.00017236304654825706 0.004674213655004137"/>
     <parent link="camera_left_link"/>
     <child link="camera_left_rgb_frame"/>

File: t2rgb_description/urdf/optimized/optimized_2023_06_07-04_04_03_PM.urdf.xacro (robot description, xacro)
@@ -23,5 +23,5 @@
   </gazebo>
   <joint name="camera_right_rgb_joint" type="fixed">
-    <origin xyz="0.003084837483015066 -0.03862858109122667 0.0012045523690927724" rpy="-0.019012904568392552 -0.007012354017393246 0.0044708591364499475"/>
+    <origin xyz="0.0030866528006126626 -0.03862892682176301 0.0012040600312779222" rpy="-0.019014307536572603 -0.007012982752457608 0.004470965879546207"/>
     <parent link="camera_right_link"/>
     <child link="camera_right_rgb_frame"/>
@@ -111,5 +111,5 @@
   </gazebo>
   <joint name="camera_left_rgb_joint" type="fixed">
-    <origin xyz="0.0016748091127418792 -0.03814222599406782 -0.006507520212859007" rpy="-0.01895612012487999 -0.007321106971785336 0.003858542386210276"/>
+    <origin xyz="0.0016760816380132545 -0.03814195476727114 -0.0065067168877275166" rpy="-0.01895617880163762 -0.007320564459510531 0.0038582082213343507"/>
     <parent link="camera_left_link"/>
     <child link="camera_left_rgb_frame"/>

File: t2rgb_description/urdf/optimized/optimized_2023_06_07-04_42_35_PM.urdf.xacro (robot description, xacro)
@@ -23,5 +23,5 @@
   </gazebo>
   <joint name="camera_right_rgb_joint" type="fixed">
-    <origin xyz="0.003084837483015066 -0.03862858109122667 0.0012045523690927724" rpy="-0.019012904568392552 -0.007012354017393246 0.0044708591364499475"/>
+    <origin xyz="0.022052578429316343 0.014453860513795993 -0.020807142677376215" rpy="0.016172472274243593 -0.0079121023625501 -0.010288794314377974"/>
     <parent link="camera_right_link"/>
     <child link="camera_right_rgb_frame"/>
@@ -111,5 +111,5 @@
   </gazebo>
   <joint name="camera_left_rgb_joint" type="fixed">
-    <origin xyz="0.0016748091127418792 -0.03814222599406782 -0.006507520212859007" rpy="-0.01895612012487999 -0.007321106971785336 0.003858542386210276"/>
+    <origin xyz="0.026223320109559373 0.014961951204945602 -0.014771998373506156" rpy="0.016260062040163382 -0.008068103061033583 -0.01089502206370241"/>
     <parent link="camera_left_link"/>
     <child link="camera_left_rgb_frame"/>

File: t2rgb_description/urdf/optimized/optimized_2023_06_07-04_48_38_PM.urdf.xacro (robot description, xacro)
@@ -23,5 +23,5 @@
   </gazebo>
   <joint name="camera_right_rgb_joint" type="fixed">
-    <origin xyz="0.003084837483015066 -0.03862858109122667 0.0012045523690927724" rpy="-0.019012904568392552 -0.007012354017393246 0.0044708591364499475"/>
+    <origin xyz="0.007238103191929118 -0.02389263449455172 -0.02933674762141532" rpy="-0.08674886945129756 -0.07363717541465754 0.0021746578403616765"/>
     <parent link="camera_right_link"/>
     <child link="camera_right_rgb_frame"/>
@@ -111,5 +111,5 @@
   </gazebo>
   <joint name="camera_left_rgb_joint" type="fixed">
-    <origin xyz="0.0016748091127418792 -0.03814222599406782 -0.006507520212859007" rpy="-0.01895612012487999 -0.007321106971785336 0.003858542386210276"/>
+    <origin xyz="0.009162703081927338 -0.02436932281882576 -0.06287351373785387" rpy="-0.08660823375480473 -0.07388345331686812 0.001259114967189536"/>
     <parent link="camera_left_link"/>
     <child link="camera_left_rgb_frame"/>

File: t2rgb_description/urdf/optimized/optimized_2023_06_07-04_52_49_PM.urdf.xacro (robot description, xacro)
@@ -23,5 +23,5 @@
   </gazebo>
   <joint name="camera_right_rgb_joint" type="fixed">
-    <origin xyz="0.003084837483015066 -0.03862858109122667 0.0012045523690927724" rpy="-0.019012904568392552 -0.007012354017393246 0.0044708591364499475"/>
+    <origin xyz="0.08610005587937627 0.029966398652179142 -0.03942459647593699" rpy="-0.15875043150088197 -0.1545292335511178 -0.1295636462388281"/>
     <parent link="camera_right_link"/>
     <child link="camera_right_rgb_frame"/>
@@ -111,5 +111,5 @@
   </gazebo>
   <joint name="camera_left_rgb_joint" type="fixed">
-    <origin xyz="0.0016748091127418792 -0.03814222599406782 -0.006507520212859007" rpy="-0.01895612012487999 -0.007321106971785336 0.003858542386210276"/>
+    <origin xyz="0.1450624507520456 0.021842275560913404 -0.09992463738699887" rpy="-0.15851360304329737 -0.1548904207475429 -0.13064995581084346"/>
     <parent link="camera_left_link"/>
     <child link="camera_left_rgb_frame"/>
